File: hardware/companions/io_jumper/io_jumper.kicad_pcb (KiCad board)
At the start: 2 copper layers, 21.9 x 51.7 mm, 12 parts, among them J1 0, J2 0, P1 PPPC202LFBN-RC, U1 MCP23008-E_SS

Commit message: Added BOM and generated gerber files
Parts:
- added DB2: RFD4d, HERMESLITE:4x1, F.Cu at (135.9, 63.1)
- R2: value 50 -> 49.9
- RF3: renamed from RF1; value BNC -> SMA
Routing:
- net GNDS: track 149.8 -> 155.1 mm
- net Net-(DB2-Pad1): track 5.08 -> 9.35 mm
- net Net-(DB2-Pad2): track 5.08 -> 9.34 mm
- net Net-(DB2-Pad3): track 5.08 -> 9.34 mm
